File: hardware/Biel_Core_One/Biel_Core_One.kicad_sch (KiCad schematic)
At the start: 0 parts

Commit message: alimentacion,proecesador y pantalla
Connections:
- no-connect marks 0 -> 2
Other:
- added sheet Alimentacion (Alimentacion.kicad_sch)
- added sheet Controles (controles.kicad_sch)
- added sheet Procesador (procesador.kicad_sch)
- added sheet pantalla (pantalla.kicad_sch)
